Commit message: 1.修改了xacro的参数，因为机器人本体变了；2.改了一些格式，加了一些打印，用来debug get switch

File: urdf/aubo_i5.xacro (robot description, xacro)
@@ -179,5 +179,5 @@
     <parent link="base_link" />
     <child link="velodyne" />
-    <origin xyz="0.32 0 0.035" rpy="0 0 3.14" />
+    <origin xyz="0.37 0 0.035" rpy="0 0 3.14" />
   </joint>
   <!--/////////////////////////////// SHOULDER_LINK ////////////////////////////////////-->
@@ -383,5 +383,5 @@
   <link name="camera_mount_link" >
     <visual>
-      <origin xyz="0.0 0.0 0.0" rpy="0 0 0"/>
+      <origin xyz="0.0 0.0 0.02" rpy="0 0 0"/>
       <geometry>
          <mesh filename="package://aubo_description/meshes/CameraMountBoard.dae" />
@@ -426,5 +426,5 @@
   <!--////////////////////////////////camera_joint/////////////////////////////////-->
   <joint name="camera_joint" type="fixed">
-    <origin xyz="0.03358 0.098 -0.05518" rpy="-1.5707 -1.5707 0"/>
+    <origin xyz="0.0160 0.098 -0.05518" rpy="-1.5707 -1.5707 0"/>
     <parent link="camera_mount_link"/>
     <child link="camera_link"/>
